File: HW_watchdog.kicad_pcb (KiCad board)
At the start: 2 copper layers, 34 x 26 mm, 19 parts, among them J1 Conn_01x02_Male, J2 Conn_01x02_Male, J3 Conn_01x02_Male, J4 Conn_01x02_Male, J5 Conn_01x02_Male, Q1 BC847, Q2 BC847, U1 ATTINY10-TS8R

Commit message: pin changed
Parts:
- J1, J2, J3, J4, J5: footprint Connector_PinHeader_1.27mm:PinHeader_1x02_P1.27mm_Vertical -> Connector_PinHeader_2.54mm:PinHeader_1x02_P2.54mm_Vertical
- moved J1 1.33 mm to (116.4, 95.7)
- moved J2 1.33 mm to (145.5, 95.7)
- moved J5 1.32 mm to (145.5, 86.6)
- moved J4 1.27 mm to (116.4, 86.7)
